Commit message: URDF: camera_tilt_link on a revolute joint about the camera servo shaft
GiaCam3A + camera module split from base_link; joint 0 = looking down,
positive = towards the nose (matches camera_tilt.py), limits -20..48.8 deg.

Co-Authored-By: Claude Opus 5.5 <noreply@anthropic.com>

File: assembly_urdf/drone_v2.urdf (robot description, URDF)
Before this commit: robot drone_v2, 5 links, 4 joints
Links:
- added link camera_tilt_link, mass 0.00914; collision box size=0.0275 0.04 0.0518; visual mesh filename=meshes/camera_tilt_link.stl
- link base_link: mass 0.74346 -> 0.73432
Joints:
- added joint camera_tilt_joint: type revolute, parent base_link, child camera_tilt_link, origin xyz=0.09525 -0.018 -0.05218 rpy=0 0 0, axis 0 -1 0, limit lower=-0.34907 upper=0.85172 effort=0.16 velocity=10.5

Commit message: URDF: camera_tilt_joint lower limit -20 -> -36 deg (grip camera angle)
Co-Authored-By: Claude Opus 5.5 <noreply@anthropic.com>

File: assembly_urdf/drone_v2.urdf (robot description, URDF)
Before this commit: robot drone_v2, 6 links, 5 joints
Joints:
- joint camera_tilt_joint: limit lower=-0.34907 upper=0.85172 effort=0.16 velocity=10.5 -> lower=-0.62832 upper=0.85172 effort=0.16 velocity=10.5

Commit message: URDF: MG90 gripper - servo horn, 2 CauNoi rods, 2 GapHang jaws (four-bar, mimic)
Assem1.SLDASM 10-25: gripper_servo_joint actuated (0 = closed toggle, -120 deg
= open), rods and jaws mimic the servo (line through exact open/closed poses,
max error 10 deg); exact four_bar() in build_meshes.py. Camera lens direction
re-read from the new assembly (CAD pose 98.2 deg); mass 0.818 kg CAD.

Co-Authored-By: Claude Opus 5.5 <noreply@anthropic.com>

File: assembly_urdf/drone_v2.urdf (robot description, URDF)
Before this commit: robot drone_v2, 6 links, 5 joints
Links:
- added link gripper_jaw_left, mass 0.01576; collision box size=0.041 0.0513 0.1372; visual mesh filename=meshes/gripper_jaw_left.stl
- added link gripper_jaw_right, mass 0.01576; collision box size=0.041 0.0513 0.1372; visual mesh filename=meshes/gripper_jaw_right.stl
- added link gripper_rod_left, mass 0.00078; visual mesh filename=meshes/gripper_rod_left.stl
- added link gripper_rod_right, mass 0.00078; visual mesh filename=meshes/gripper_rod_right.stl
- added link gripper_servo_link, mass 0.00053; visual mesh filename=meshes/gripper_servo_link.stl
- link base_link: mass 0.73432 -> 0.75082
Joints:
- added joint gripper_jaw_left_joint: type revolute, parent base_link, child gripper_jaw_left, origin xyz=0.0025 0.03151 -0.0625 rpy=0 0 0, axis 1 0 0, limit lower=0 upper=0.73339 effort=1 velocity=10, mimic joint=gripper_servo_joint multiplier=-0.3502 offset=0
- added joint gripper_jaw_right_joint: type revolute, parent base_link, child gripper_jaw_right, origin xyz=0.0025 -0.0315 -0.0625 rpy=0 0 0, axis 1 0 0, limit lower=-0.58991 upper=0 effort=1 velocity=10, mimic joint=gripper_servo_joint multiplier=0.2817 offset=0
- added joint gripper_rod_left_joint: type revolute, parent gripper_servo_link, child gripper_rod_left, origin xyz=0 -0.00927 -0.00008 rpy=0 0 0, axis 1 0 0, limit lower=0 upper=2.08298 effort=1 velocity=20, mimic joint=gripper_servo_joint multiplier=-0.9945 offset=0
- added joint gripper_rod_right_joint: type revolute, parent gripper_servo_link, child gripper_rod_right, origin xyz=0 0.00927 0.00007 rpy=0 0 0, axis 1 0 0, limit lower=0 upper=1.78045 effort=1 velocity=20, mimic joint=gripper_servo_joint multiplier=-0.8501 offset=0
- added joint gripper_servo_joint: type revolute, parent base_link, child gripper_servo_link, origin xyz=-0.00225 0 -0.08462 rpy=0 0 0, axis 1 0 0, limit lower=-2.0944 upper=0 effort=0.18 velocity=10.5

Commit message: URDF gripper: open = -180 deg (full MG90 travel, second toggle, jaws 56 deg)
Kept open whenever not gripping so the fingers stay 45 mm above the leg plane;
no body contact over 0..-180 deg. Rod angles kept continuous past 180 deg.

Co-Authored-By: Claude Opus 5.5 <noreply@anthropic.com>

File: assembly_urdf/drone_v2.urdf (robot description, URDF)
Before this commit: robot drone_v2, 11 links, 10 joints
Joints:
- joint gripper_jaw_left_joint: limit lower=0 upper=0.73339 effort=1 velocity=10 -> lower=0 upper=0.97716 effort=1 velocity=10; mimic joint=gripper_servo_joint multiplier=-0.3502 offset=0 -> joint=gripper_servo_joint multiplier=-0.3110 offset=0
- joint gripper_jaw_right_joint: limit lower=-0.58991 upper=0 effort=1 velocity=10 -> lower=-0.97425 upper=0 effort=1 velocity=10; mimic joint=gripper_servo_joint multiplier=0.2817 offset=0 -> joint=gripper_servo_joint multiplier=0.3101 offset=0
- joint gripper_rod_left_joint: limit lower=0 upper=2.08298 effort=1 velocity=20 -> lower=0 upper=3.41901 effort=1 velocity=20; mimic joint=gripper_servo_joint multiplier=-0.9945 offset=0 -> joint=gripper_servo_joint multiplier=-1.0883 offset=0
- joint gripper_rod_right_joint: limit lower=0 upper=1.78045 effort=1 velocity=20 -> lower=0 upper=2.85854 effort=1 velocity=20; mimic joint=gripper_servo_joint multiplier=-0.8501 offset=0 -> joint=gripper_servo_joint multiplier=-0.9099 offset=0
- joint gripper_servo_joint: limit lower=-2.0944 upper=0 effort=0.18 velocity=10.5 -> lower=-3.14159 upper=0 effort=0.18 velocity=10.5
